File: schematic/opti_filmscanner.kicad_sch (KiCad schematic)
At the start: 5 parts, among them SW1 SW_Push

Commit message: expanded readme
Other:
- note added: "EndStop"
- note removed: "Push BTN not necessary"
Changed lines of the file:
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@@
     (stroke (width 0) (type default) (color 0 0 0 0))
   )
-  (text "Push BTN not necessary" (at 120.65 88.9 0)
+  (text "EndStop" (at 123.19 88.9 0)
     (effects (font (size 1.27 1.27)) (justify left bottom))
   )
